Commit message: Add onshape to robot config for custom arm, change from panda arm to custom arm

File: src/arm_description/urdf/arm.urdf (robot description, URDF)
Before this commit: robot arm, 13 links, 12 joints
Links:
- removed link arm_hand
- removed link arm_hand_tcp
- removed link arm_leftfinger
- removed link arm_link0
- removed link arm_link1
- removed link arm_link2
- removed link arm_link3
- removed link arm_link4
- removed link arm_link5
- removed link arm_link6
- removed link arm_link7
- removed link arm_link8
- removed link arm_rightfinger
- added link base_link, mass 0.357273; collision mesh filename=package://arm_description/assets/base.stl; collision mesh filename=package://arm_description/assets/servo_base.stl
- added link link_1, mass 0.3873; collision mesh filename=package://arm_description/assets/base_cover.stl; collision mesh filename=package://arm_description/assets/hex_nut_grade_a___b_m4x0_7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
- added link link_2, mass 0.00888911; collision mesh filename=package://arm_description/assets/6mm_bearing_v2.stl; collision mesh filename=package://arm_description/assets/6mm_bearing_v2.stl
- added link link_3, mass 0.00639747; collision mesh filename=package://arm_description/assets/hex_nut_grade_a___b_m2x0_4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; collision mesh filename=package://arm_description/assets/hex_nut_grade_a___b_m2x0_4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
- added link link_4, mass 0.00530132; collision mesh filename=package://arm_description/assets/6mm_bearing_v2.stl; collision mesh filename=package://arm_description/assets/hex_nut_grade_a___b_m2x0_4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
- added link link_5, mass 0.00530132; collision mesh filename=package://arm_description/assets/6mm_bearing_v2.stl; collision mesh filename=package://arm_description/assets/hex_nut_grade_a___b_m2x0_4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
- added link link_6, mass 1e-09; collision mesh filename=package://arm_description/assets/wheel_gear_v6__2.stl; visual mesh filename=package://arm_description/assets/wheel_gear_v6__2.stl
- added link tcp, mass 1e-9
Joints:
- removed joint arm_finger_joint1
- removed joint arm_finger_joint2
- removed joint arm_hand_joint
- removed joint arm_hand_tcp_joint
- removed joint arm_joint1
- removed joint arm_joint2
- removed joint arm_joint3
- removed joint arm_joint4
- removed joint arm_joint5
- removed joint arm_joint6
- removed joint arm_joint7
- removed joint arm_joint8
- added joint joint_1: type revolute, parent base_link, child link_1, origin xyz=1.54081e-17 9.14136e-05 0.0755 rpy=-3.14159 -3.6506e-16 -3.10006, axis 0 0 1, limit lower=-3.10006 upper=1.61232 effort=10 velocity=1
- added joint joint_2: type revolute, parent link_1, child link_2, origin xyz=-2.24205e-17 0.0315746 -0.0675 rpy=1.5708 -1.5708 0, axis 0 0 1, limit lower=-1.5708 upper=1.5708 effort=10 velocity=1
- added joint joint_3: type revolute, parent link_2, child link_3, origin xyz=-0.166 -1.91133e-18 -2.08167e-16 rpy=3.14159 -8.28144e-16 -1.5708, axis 0 0 1, limit lower=-1.5708 upper=1.5708 effort=10 velocity=1
- added joint joint_4: type revolute, parent link_3, child link_4, origin xyz=-1.83989e-15 0.224 -4.16334e-16 rpy=-3.14159 -8.69067e-16 -1.5708, axis 0 0 1, limit lower=-1.5708 upper=1.5708 effort=10 velocity=1
- added joint joint_5: type revolute, parent link_4, child link_5, origin xyz=-0.095 0.0315 0.03175 rpy=1.5708 -5.58182e-14 1.16592e-14, axis 0 0 1, limit lower=0 upper=3.14159 effort=10 velocity=1
- added joint joint_6: type revolute, parent link_5, child link_6, origin xyz=-0.095 0.0315 0.03175 rpy=1.5708 1.5708 0, axis 0 0 1, limit lower=0 upper=4.71239 effort=10 velocity=1
- added joint tcp_frame: type fixed, parent link_6, child tcp, origin xyz=1.0842e-19 0 0.0005 rpy=3.14159 -4.48041e-19 0, axis 0 0 0

File: src/arm_description/urdf/arm_ros2_control.xacro (robot description, xacro)
@@ -7,44 +7,34 @@
             <param name="fake_sensor_commands">false</param>
         </hardware>
-        <joint name="arm_joint1">
+        <joint name="joint_1">
             <command_interface name="position"/>
             <state_interface name="position"/>
             <param name="servo_id">0</param>
         </joint>
-        <joint name="arm_joint2">
+        <joint name="joint_2">
             <command_interface name="position"/>
             <state_interface name="position"/>
             <param name="servo_id">1</param>
         </joint>
-        <joint name="arm_joint3">
+        <joint name="joint_3">
             <command_interface name="position"/>
             <state_interface name="position"/>
             <param name="servo_id">2</param>
         </joint>
-        <joint name="arm_joint4">
+        <joint name="joint_4">
             <command_interface name="position"/>
             <state_interface name="position"/>
             <param name="servo_id">3</param>
         </joint>
-        <joint name="arm_joint5">
+        <joint name="joint_5">
             <command_interface name="position"/>
             <state_interface name="position"/>
             <param name="servo_id">4</param>
         </joint>
-        <joint name="arm_joint6">
+        <joint name="joint_6">
             <command_interface name="position"/>
             <state_interface name="position"/>
             <param name="servo_id">5</param>
         </joint>
-        <joint name="arm_joint7">
-            <command_interface name="position"/>
-            <state_interface name="position"/>
-            <param name="servo_id">6</param>
-        </joint>
-        <joint name="arm_finger_joint1">
-            <command_interface name="position"/>
-            <state_interface name="position"/>
-            <param name="servo_id">7</param>
-        </joint>
     </ros2_control>
     </xacro:macro>

Commit message: update urdf

File: src/arm_description/urdf/arm.urdf (robot description, URDF)
Before this commit: robot arm, 8 links, 7 joints
Links:
- link base_link: mass 0.357273 -> 0.00490817; geometry collision mesh filename=package://arm_description/assets/base.stl; collision mesh filename=package://arm_description/assets/pca9685_v18.stl
- link link_1: mass 0.3873 -> 0.373149; geometry collision mesh filename=package://arm_description/assets/base_cover.stl; collision mesh filename=package://arm_description/assets/joint_2_connecter.stl
- link link_2: mass 0.00888911 -> 0.014882; geometry collision mesh filename=package://arm_description/assets/6mm_bearing_v2.stl; collision mesh filename=package://arm_description/assets/6mm_bearing_v2.stl
- link link_3: mass 0.00639747 -> 0.0138515; geometry collision mesh filename=package://arm_description/assets/link__rotation_default_len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; collision mesh filename=package://arm_description/assets/servo_base__2.stl
- link link_4: mass 0.00530132 -> 0.00854202; geometry collision mesh filename=package://arm_description/assets/6mm_bearing_v2.stl; collision mesh filename=package://arm_description/assets/large_support.stl
- link link_5: mass 0.00530132 -> 0.00854202; geometry collision mesh filename=package://arm_description/assets/6mm_bearing_v2.stl; collision mesh filename=package://arm_description/assets/large_support.stl
Joints:
- joint joint_1: limit lower=-3.10006 upper=1.61232 effort=10 velocity=1 -> lower=0 upper=3.14159 effort=10 velocity=1; origin xyz=1.54081e-17 9.14136e-05 0.0755 rpy=-3.14159 -3.6506e-16 -3.10006 -> xyz=1.20311e-16 9.14136e-05 0.0755 rpy=-3.14159 1.3935e-15 -2.22045e-16
- joint joint_2: limit lower=-1.5708 upper=1.5708 effort=10 velocity=1 -> lower=0 upper=3.14159 effort=10 velocity=1; origin xyz=-2.24205e-17 0.0315746 -0.0675 rpy=1.5708 -1.5708 0 -> xyz=-2.9121e-17 0.0315746 -0.0675 rpy=1.5708 4.44089e-16 -3.14159
- joint joint_3: limit lower=-1.5708 upper=1.5708 effort=10 velocity=1 -> lower=0 upper=3.14159 effort=10 velocity=1; origin xyz=-0.166 -1.91133e-18 -2.08167e-16 rpy=3.14159 -8.28144e-16 -1.5708 -> xyz=-0.166 -2.77556e-17 -1.45717e-16 rpy=-3.14159 -4.14819e-16 1.08368e-25
- joint joint_4: limit lower=-1.5708 upper=1.5708 effort=10 velocity=1 -> lower=0 upper=3.14159 effort=10 velocity=1; origin xyz=-1.83989e-15 0.224 -4.16334e-16 rpy=-3.14159 -8.69067e-16 -1.5708 -> xyz=1.11022e-16 0.224 -8.32667e-17 rpy=1.05083e-15 4.0358e-16 4.996e-16
- joint joint_5: origin xyz=-0.095 0.0315 0.03175 rpy=1.5708 -5.58182e-14 1.16592e-14 -> xyz=0.095 -0.0315 0.03175 rpy=-1.5708 1.5708 0
- joint tcp_frame: origin xyz=1.0842e-19 0 0.0005 rpy=3.14159 -4.48041e-19 0 -> xyz=-5.55112e-17 -1.38778e-17 0.0005 rpy=-3.14159 4.22164e-31 -9.5309e-30

Commit message: update urdf

File: src/arm_description/urdf/arm.urdf (robot description, URDF)
Before this commit: robot arm, 8 links, 7 joints
Links:
- link base_link: mass 0.00490817 -> 0.0051027
- link link_1: mass 0.373149 -> 0.368704; geometry collision mesh filename=package://arm_description/assets/base_cover.stl; collision mesh filename=package://arm_description/assets/joint_2_connecter1.stl
- link link_5: mass 0.00854202 -> 0.0143668; geometry collision mesh filename=package://arm_description/assets/6mm_bearing_v2.stl; collision mesh filename=package://arm_description/assets/large_support.stl
Joints:
- joint joint_1: limit lower=0 upper=3.14159 effort=10 velocity=1 -> lower=-1.7299 upper=1.4117 effort=10 velocity=1; origin xyz=1.20311e-16 9.14136e-05 0.0755 rpy=-3.14159 1.3935e-15 -2.22045e-16 -> xyz=-2.23802e-17 9.14136e-05 0.0755 rpy=3.14159 -8.32667e-16 -1.7299
- joint joint_2: limit lower=0 upper=3.14159 effort=10 velocity=1 -> lower=-0.0528179 upper=3.08877 effort=10 velocity=1; origin xyz=-2.9121e-17 0.0315746 -0.0675 rpy=1.5708 4.44089e-16 -3.14159 -> xyz=-8.63296e-18 0.0315746 -0.0675 rpy=1.5708 -0.0528179 3.14159
- joint joint_3: limit lower=0 upper=3.14159 effort=10 velocity=1 -> lower=-0.947497 upper=2.1941 effort=10 velocity=1; origin xyz=-0.166 -2.77556e-17 -1.45717e-16 rpy=-3.14159 -4.14819e-16 1.08368e-25 -> xyz=-0.166 1.66533e-16 -2.70617e-16 rpy=-3.14159 -4.14511e-16 3.96651e-18
- joint joint_4: limit lower=0 upper=3.14159 effort=10 velocity=1 -> lower=-0.114869 upper=3.02672 effort=10 velocity=1; origin xyz=1.11022e-16 0.224 -8.32667e-17 rpy=1.05083e-15 4.0358e-16 4.996e-16 -> xyz=-0.181878 0.130753 -6.45317e-16 rpy=-2.62547e-15 -2.40252e-15 0.947497
- joint joint_5: limit lower=0 upper=3.14159 effort=10 velocity=1 -> lower=-2.33032 upper=0.81127 effort=10 velocity=1; origin xyz=0.095 -0.0315 0.03175 rpy=-1.5708 1.5708 0 -> xyz=0.0979844 -0.0204038 0.03175 rpy=1.5708 -0.759527 -3.02672
- joint joint_6: limit lower=0 upper=4.71239 effort=10 velocity=1 -> lower=-0.00948244 upper=4.70291 effort=10 velocity=1; origin xyz=-0.095 0.0315 0.03175 rpy=1.5708 1.5708 0 -> xyz=-0.145 0.0315 0.03175 rpy=1.5708 1.56131 -6.00447e-13
- joint tcp_frame: origin xyz=-5.55112e-17 -1.38778e-17 0.0005 rpy=-3.14159 4.22164e-31 -9.5309e-30 -> xyz=0 0 0.0005 rpy=-3.14159 -2.36422e-17 -7.48843e-17

Commit message: update urdf

File: src/arm_description/urdf/arm.urdf (robot description, URDF)
Before this commit: robot arm, 8 links, 7 joints
Links:
- link link_1: mass 0.368704 -> 0.336956
- link link_4: mass 0.00854202 -> 0.0143668; geometry collision mesh filename=package://arm_description/assets/6mm_bearing_v2.stl; collision mesh filename=package://arm_description/assets/large_support.stl
- link link_5: geometry collision mesh filename=package://arm_description/assets/6mm_bearing_v2.stl; collision mesh filename=package://arm_description/assets/large_support.stl
- link link_6: mass 1e-09 -> 0.00249164; geometry collision mesh filename=package://arm_description/assets/6mm_bearing_v2__2.stl; collision mesh filename=package://arm_description/assets/large_support__2.stl
Joints:
- joint joint_1: limit lower=-1.7299 upper=1.4117 effort=10 velocity=1 -> lower=3.55187e-14 upper=3.14159 effort=10 velocity=1; origin xyz=-2.23802e-17 9.14136e-05 0.0755 rpy=3.14159 -8.32667e-16 -1.7299 -> xyz=1.39768e-18 9.14136e-05 0.0755 rpy=1.7878e-15 -9.97279e-17 3.14159
- joint joint_2: limit lower=-0.0528179 upper=3.08877 effort=10 velocity=1 -> lower=-1.26017e-14 upper=3.14159 effort=10 velocity=1; origin xyz=-8.63296e-18 0.0315746 -0.0675 rpy=1.5708 -0.0528179 3.14159 -> xyz=-1.85992e-17 -0.0315746 0.0675 rpy=-1.5708 1.26492e-14 -3.14159
- joint joint_3: limit lower=-0.947497 upper=2.1941 effort=10 velocity=1 -> lower=-1.98875e-14 upper=3.14159 effort=10 velocity=1; origin xyz=-0.166 1.66533e-16 -2.70617e-16 rpy=-3.14159 -4.14511e-16 3.96651e-18 -> xyz=-0.166 -2.77556e-17 -2.08167e-17 rpy=-3.14159 2.92704e-17 5.55112e-17
- joint joint_4: limit lower=-0.114869 upper=3.02672 effort=10 velocity=1 -> lower=7.28578e-15 upper=3.14159 effort=10 velocity=1; origin xyz=-0.181878 0.130753 -6.45317e-16 rpy=-2.62547e-15 -2.40252e-15 0.947497 -> xyz=-3.66374e-15 0.224 0.063 rpy=1.3247e-15 -5.66554e-16 -3.14159
- joint joint_5: limit lower=-2.33032 upper=0.81127 effort=10 velocity=1 -> lower=-3.55187e-14 upper=3.14159 effort=10 velocity=1; origin xyz=0.0979844 -0.0204038 0.03175 rpy=1.5708 -0.759527 -3.02672 -> xyz=-0.145 -0.0315 -0.03175 rpy=1.5708 1.5708 0
- joint joint_6: limit lower=-0.00948244 upper=4.70291 effort=10 velocity=1 -> lower=0 upper=3.14159 effort=10 velocity=1; origin xyz=-0.145 0.0315 0.03175 rpy=1.5708 1.56131 -6.00447e-13 -> xyz=-0.175 -0.0315 -0.03175 rpy=1.5708 1.5708 0
- joint tcp_frame: origin xyz=0 0 0.0005 rpy=-3.14159 -2.36422e-17 -7.48843e-17 -> xyz=-0.033 2.498e-16 -0.03175 rpy=3.14159 1.5708 0

Commit message: update urdf

File: src/arm_description/urdf/arm.urdf (robot description, URDF)
Before this commit: robot arm, 8 links, 7 joints
Joints:
- joint joint_1: limit lower=3.55187e-14 upper=3.14159 effort=10 velocity=1 -> lower=0 upper=3.14159 effort=10 velocity=1
- joint joint_2: limit lower=-1.26017e-14 upper=3.14159 effort=10 velocity=1 -> lower=0 upper=3.14159 effort=10 velocity=1; origin xyz=-1.85992e-17 -0.0315746 0.0675 rpy=-1.5708 1.26492e-14 -3.14159 -> xyz=-1.89511e-17 -0.0315746 0.0675 rpy=-1.5708 -1.27563e-14 -3.14159
- joint joint_3: limit lower=-1.98875e-14 upper=3.14159 effort=10 velocity=1 -> lower=-4.44089e-15 upper=3.14159 effort=10 velocity=1; origin xyz=-0.166 -2.77556e-17 -2.08167e-17 rpy=-3.14159 2.92704e-17 5.55112e-17 -> xyz=-0.166 0 -1.38778e-17 rpy=3.14159 5.80243e-15 0
- joint joint_4: limit lower=7.28578e-15 upper=3.14159 effort=10 velocity=1 -> lower=0 upper=3.14159 effort=10 velocity=1; origin xyz=-3.66374e-15 0.224 0.063 rpy=1.3247e-15 -5.66554e-16 -3.14159 -> xyz=3.33067e-16 0.224 0.063 rpy=1.33151e-14 -4.56336e-15 -3.14159
- joint joint_5: limit lower=-3.55187e-14 upper=3.14159 effort=10 velocity=1 -> lower=0 upper=3.14159 effort=10 velocity=1
- joint tcp_frame: origin xyz=-0.033 2.498e-16 -0.03175 rpy=3.14159 1.5708 0 -> xyz=-0.033 5.55112e-17 -0.03175 rpy=-3.14159 1.5708 0

Commit message: increase joint velocity limits, add arm_execution_manager for planning. operator no longer supports controller, only poses from hand gestures

File: src/arm_description/urdf/arm.urdf (robot description, URDF)
Before this commit: robot arm, 8 links, 7 joints
Joints:
- joint joint_1: limit lower=0 upper=3.14159 effort=10 velocity=1 -> lower=0 upper=3.14159 effort=10 velocity=2
- joint joint_2: limit lower=0 upper=3.14159 effort=10 velocity=1 -> lower=0 upper=3.14159 effort=10 velocity=2
- joint joint_3: limit lower=-4.44089e-15 upper=3.14159 effort=10 velocity=1 -> lower=-4.44089e-15 upper=3.14159 effort=10 velocity=2
- joint joint_4: limit lower=0 upper=3.14159 effort=10 velocity=1 -> lower=0 upper=3.14159 effort=10 velocity=2
- joint joint_5: limit lower=0 upper=3.14159 effort=10 velocity=1 -> lower=0 upper=3.14159 effort=10 velocity=2
- joint joint_6: limit lower=0 upper=3.14159 effort=10 velocity=1 -> lower=0 upper=3.14159 effort=10 velocity=2
